File: Polemo Core/Polemo Core 2/Polemo Core 2.kicad_sch (KiCad schematic)
At the start: 174 parts, among them P1 Header-Male-2.54_2x2, P2 Header-Male-2.54_2x2, Q1 BC847_C2910145, Q2 MMBT5551LT1G, Q3 AO3401A, Q4 AO3401A, Q5 MMBT5551LT1G, U1 ATSAML21G18B-AUT, U10 74LVC1G08GV,125, U11 LT3014BHVES5#TRMPBF, U12 TXU0202DCUR, U13 TLV7031DBVR, U14 TLR341G-GTR, U15 803-87-006-10-001101, U2 XC6209F332MR-G, U3 MC14043BDR2G, U4 LMV793MFX/NOPB, U5 TPS7A2030PDBVR, U6 TLV3201AIDBVT, U7 OPA357AIDBVR, U8 TLR341G-GTR, U9 MF-ASML020/6-2, X1 32.768kHz

Commit message: Refactor code structure for improved readability and maintainability
Connections:
- net 3V3: no longer R27.1, U10.4 (Y)
- new net: R27.1, U10.4 (Y)
Other:
- company: Safecast -> (none)
- title: bGeigieScint -> (none)
Changed lines of the file:
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@@
 	(paper "A2")
 	(title_block
-		(title "bGeigieScint")
 		(date "2025-11-23")
-		(rev "1.3")
-		(company "Safecast")
 	)
 	(text "3V3"
@@
 	)
 	(junction
-		(at 378.46 363.22)
-		(diameter 0)
-		(color 0 0 0 0)
-	)
-	(junction
 		(at 410.21 349.25)
 		(diameter 0)
@@
 	(wire
 		(pts
-			(xy 444.5 373.38) (xy 444.5 363.22)
+			(xy 443.865 356.235) (xy 443.865 373.38)
 		)
 		(stroke
@@
 	(wire
 		(pts
-			(xy 378.46 363.22) (xy 342.9 363.22)
-		)
-		(stroke
-			(width 0)
-			(type default)
-		)
-	)
-	(wire
-		(pts
 			(xy 378.46 39.37) (xy 378.46 57.15)
 		)
@@
 	(wire
 		(pts
-			(xy 444.5 363.22) (xy 378.46 363.22)
+			(xy 443.865 373.38) (xy 431.8 373.38)
 		)
 		(stroke
@@
 	(wire
 		(pts
-			(xy 431.8 373.38) (xy 444.5 373.38)
-		)
-		(stroke
-			(width 0)
-			(type default)
-		)
-	)
-	(wire
-		(pts
 			(xy 482.6 327.66) (xy 494.03 327.66)
 		)
@@
 	(wire
 		(pts
-			(xy 342.9 339.09) (xy 346.71 339.09)
+			(xy 343.535 339.09) (xy 346.71 339.09)
 		)
 		(stroke
@@
 	(wire
 		(pts
+			(xy 343.535 356.235) (xy 443.865 356.235)
+		)
+		(stroke
+			(width 0)
+			(type default)
+		)
+	)
+	(wire
+		(pts
 			(xy 190.5 345.44) (xy 190.5 349.25)
 		)
@@
 	(wire
 		(pts
-			(xy 342.9 363.22) (xy 342.9 339.09)
+			(xy 343.535 356.235) (xy 343.535 339.09)
 		)
 		(stroke
