File: bGeigieScint/bGeigieScint.kicad_sch (KiCad schematic)
At the start: 174 parts, among them P1 Header-Male-2.54_2x2, P2 Header-Male-2.54_2x2, Q1 BC847_C2910145, Q2 MMBT5551LT1G, Q3 AO3401A, Q4 AO3401A, Q5 MMBT5551LT1G, U1 ATSAML21G18B-AUT, U10 74LVC1G08GV,125, U11 LT3014BHVES5#TRMPBF, U12 TXU0202DCUR, U13 TLV7031DBVR, U14 TLR341G-GTR, U15 803-87-006-10-001101, U2 XC6209F332MR-G, U3 MC14043BDR2G, U4 LMV793MFX/NOPB, U5 TPS7A2030PDBVR, U6 TLV3201AIDBVT, U7 OPA357AIDBVR, U8 TLR341G-GTR, U9 MF-ASML020/6-2, X1 32.768kHz

Commit message: feat: Migrate processor from SAML21G18B to ESP32-C3-MINI-1
Replace Microchip SAML21G18B with Espressif ESP32-C3-MINI-1 module for
lower power consumption and WiFi/BLE connectivity.

Hardware changes:
- Update KiCad schematic symbol from ATSAML21G18B-AUT to ESP32-C3-MINI-1-N4
- Change footprint from QFN-48 to ESP32-C3-MINI-1 module footprint
- Update component properties (manufacturer, part number, LCSC supplier code)

Firmware configuration:
- Replace atmelsam platform with espressif32 in platformio.ini
- Configure for ESP32-C3-DEVKITM-1 board with Arduino framework
- Set CPU frequency to 160MHz, 4MB flash
- Enable USB CDC for serial communication
- Remove all SAML21-specific ASF framework dependencies

Note: Pin connections in schematic need manual rewiring in KiCad.
Firmware code requires complete rewrite from ASF to Arduino/ESP-IDF APIs.

🤖 Generated with [Claude Code](https://claude.com/claude-code)

Co-Authored-By: Claude Sonnet 4.5 <noreply@anthropic.com>
Parts:
- U1: value ATSAML21G18B-AUT -> ESP32-C3-MINI-1; footprint Package_DFN_QFN:QFN-48-1EP_7x7mm_P0.5mm_EP5.15x5.15mm -> RF_Module:ESP32-C3-MINI-1; symbol ATSAML21G18B-AUT -> ESP32-C3-MINI-1; Manufacturer MICROCHIP(美国微芯) -> Espressif Systems; Manufacturer Part ATSAML21G18B-AUT -> ESP32-C3-MINI-1-N4; Supplier Part C2052742 -> C5180825
Changed lines of the file:
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@@
 	)
 	(symbol
-		(lib_id "ATSAML21G18B-AUT")
+		(lib_id "ESP32-C3-MINI-1")
 		(at 299.72 158.75 0)
 		(unit 0)
@@
 			)
 		)
-		(property "Value" "ATSAML21G18B-AUT"
+		(property "Value" "ESP32-C3-MINI-1"
 			(at 297.942 124.4727 0)
 			(effects
@@
 			)
 		)
-		(property "Footprint" "Package_DFN_QFN:QFN-48-1EP_7x7mm_P0.5mm_EP5.15x5.15mm"
+		(property "Footprint" "RF_Module:ESP32-C3-MINI-1"
 			(at 299.72 158.75 0)
 			(effects
@@
 			)
 		)
-		(property "Manufacturer Part" "ATSAML21G18B-AUT"
+		(property "Manufacturer Part" "ESP32-C3-MINI-1-N4"
 			(at 299.72 158.75 0)
 			(effects
@@
 			)
 		)
-		(property "Manufacturer" "MICROCHIP(美国微芯)"
+		(property "Manufacturer" "Espressif Systems"
 			(at 299.72 158.75 0)
 			(effects
@@
 			)
 		)
-		(property "Supplier Part" "C2052742"
+		(property "Supplier Part" "C5180825"
 			(at 299.72 158.75 0)
 			(effects

Commit message: feat: Switch from ESP32-C3-MINI-1 module to ESP32-C3 Super Mini board
Replace ESP32-C3-MINI-1 surface-mount module with ESP32-C3 Super Mini
development board as a plug-in module for easier prototyping and
replacement.

Hardware changes:
- Update KiCad symbol from ESP32-C3-MINI-1 to ESP32-C3-SuperMini
- Change footprint from RF module to 2x8 pin header (2.54mm pitch)
- Update component properties for generic/OEM sourcing

Benefits:
- Easier prototyping and testing
- Replaceable module (no soldering ESP32 chip)
- Built-in USB-C, voltage regulator, and programming circuitry
- Compact form factor (16 pins, 11 GPIOs available)

Note: Pin connections in schematic still need manual rewiring to match
Super Mini pinout (GPIO0-10, GPIO20-21).

🤖 Generated with [Claude Code](https://claude.com/claude-code)

Co-Authored-By: Claude Sonnet 4.5 <noreply@anthropic.com>
Parts:
- U1: symbol ESP32-C3-MINI-1 -> ESP32-C3-SuperMini
Other:
- moved on the sheet: H2, H3, R43, R44, R45, R46, R47, R48, R49, R50, R51, R52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

Commit message: fix: Update ESP32-C3 Super Mini instance properties in schematic
Complete the migration by updating the component instance properties
that were missed in the previous commit. The symbol definition was
updated but the placed component instance still had old values.

Changes:
- Update component value to ESP32-C3-SuperMini
- Update footprint to PinHeader_2x08_P2.54mm_Vertical
- Update manufacturer part to "ESP32-C3 Super Mini"
- Update manufacturer to "Generic/OEM"
- Update supplier part to "Various"

🤖 Generated with [Claude Code](https://claude.com/claude-code)

Co-Authored-By: Claude Sonnet 4.5 <noreply@anthropic.com>
Parts:
- U1: value ESP32-C3-MINI-1 -> ESP32-C3-SuperMini; footprint RF_Module:ESP32-C3-MINI-1 -> Connector_PinHeader_2.54mm:PinHeader_2x08_P2.54mm_Vertical; Manufacturer Espressif Systems -> Generic/OEM; Manufacturer Part ESP32-C3-MINI-1-N4 -> ESP32-C3 Super Mini; Supplier Part C5180825 -> Various
Changed lines of the file:
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@@
 			)
 		)
-		(property "Value" "ESP32-C3-MINI-1"
+		(property "Value" "ESP32-C3-SuperMini"
 			(at 297.942 124.4727 0)
 			(effects
@@
 			)
 		)
-		(property "Footprint" "RF_Module:ESP32-C3-MINI-1"
+		(property "Footprint" "Connector_PinHeader_2.54mm:PinHeader_2x08_P2.54mm_Vertical"
 			(at 299.72 158.75 0)
 			(effects
@@
 			)
 		)
-		(property "Manufacturer Part" "ESP32-C3-MINI-1-N4"
+		(property "Manufacturer Part" "ESP32-C3 Super Mini"
 			(at 299.72 158.75 0)
 			(effects
@@
 			)
 		)
-		(property "Manufacturer" "Espressif Systems"
+		(property "Manufacturer" "Generic/OEM"
 			(at 299.72 158.75 0)
 			(effects
@@
 			)
 		)
-		(property "Supplier Part" "C5180825"
+		(property "Supplier Part" "Various"
 			(at 299.72 158.75 0)
 			(effects

Commit message: fix: Replace 48-pin SAML21 symbol with correct 16-pin ESP32-C3 Super Mini
Completely redesign the symbol to match the actual ESP32-C3 Super Mini
board pinout with only 16 pins instead of the 48 pins from SAML21.

Pin layout (2x8 header):
Left side:  GND, 3V3, GPIO0-5
Right side: GPIO6-10, GPIO20-21, GND

Changes:
- Remove all 48 SAML21 pins (PA00-PA31, PB00-PB23, etc.)
- Add 16 pins matching ESP32-C3 Super Mini actual pinout
- Adjust symbol size to fit 16-pin layout
- Maintain 2.54mm pin spacing for standard headers

Stats: -888 lines, +301 lines (symbol simplified)

🤖 Generated with [Claude Code](https://claude.com/claude-code)

Co-Authored-By: Claude Sonnet 4.5 <noreply@anthropic.com>
Connections:
- net 3V3: no longer U1.17 (VDDIO), U1.36 (VDDIO), U1.44 (VDDIN)
- net GND: no longer U1.18 (GND), U1.35 (GND), U1.42 (GND), U1.5 (GNDANA)
- net PA02_DAC_HV: no longer U1.3 (PA02)
- net PA03_RAMP_EN: no longer U1.4 (PA03)
- net PA04_RAMP_OUT: no longer U1.9 (PA04)
- net PA05_DAC_THR: no longer U1.10 (PA05)
- net PA06: no longer U1.11 (PA06)
- net PA07_PEAKDET_OUT: no longer U1.12 (PA07)
- net PA08_RESET: no longer U1.13 (PA08)
- net PA09: no longer U1.14 (PA09)
- net PA10_PWM: no longer U1.15 (PA10)
- net PA11_RAMP_TRG: no longer U1.16 (PA11)
- net PA12_TX: no longer U1.21 (PA12)
- net PA13_RX: no longer U1.22 (PA13)
- net PA14_AFE_EN: no longer U1.23 (PA14)
- net PA15_PEAKDET_DISABLE: no longer U1.24 (PA15)
- net PA16_SDA: no longer U1.25 (PA16)
- net PA17_SCL: no longer U1.26 (PA17)
- net PA18_TRG_OUT: no longer U1.27 (PA18)
- net PA20: no longer U1.29 (PA20)
- net PA21: no longer U1.30 (PA21)
- net PA22: no longer U1.31 (PA22)
- net PA23_TRG_OUT: no longer U1.32 (PA23)
- net PB02: no longer U1.47 (PB02)
- net PB03_PEAKDET_EN: no longer U1.48 (PB03)
- net PB08: no longer U1.7 (PB08)
- net PB09: no longer U1.8 (PB09)
- net PB10_HV_COMP_OUT: no longer U1.19 (PB10)
- net PB11: no longer U1.20 (PB11)
- net PB22: no longer U1.37 (PB22)
- net PB23: no longer U1.38 (PB23)
- net RESET: no longer U1.40 (RESET#)
- net SWDCLK: no longer U1.45 (PA30)
- net SWDIO: no longer U1.46 (PA31)
- net USBDN: no longer U1.33 (PA24)
- net USBDP: no longer U1.34 (PA25)
- net USBVBUS: no longer U1.39 (PA27)
- net at C48.2, C49.2, C50.2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: no longer U1.6 (VDDANA)
- net at C43.2, X1.2: no longer U1.1 (PA00)
- net at C42.2, X1.1: no longer U1.2 (PA01)
- net at LED1.1 (C): no longer U1.28 (PA19)
- net at C45.2: no longer U1.41 (VDDCORE)
