File: bGeigieScint/bGeigieScint.kicad_sch (KiCad schematic)
At the start: 174 parts, among them P1 Header-Male-2.54_2x2, P2 Header-Male-2.54_2x2, Q1 BC847_C2910145, Q2 MMBT5551LT1G, Q3 AO3401A, Q4 AO3401A, Q5 MMBT5551LT1G, U1 ESP32-C3-SuperMini, U10 74LVC1G08GV,125, U11 LT3014BHVES5#TRMPBF, U12 TXU0202DCUR, U13 TLV7031DBVR, U14 TLR341G-GTR, U15 803-87-006-10-001101, U2 XC6209F332MR-G, U3 MC14043BDR2G, U4 LMV793MFX/NOPB, U5 TPS7A2030PDBVR, U6 TLV3201AIDBVT, U7 OPA357AIDBVR, U8 TLR341G-GTR, U9 MF-ASML020/6-2, X1 32.768kHz

Commit message: Progress  on switching the ESP32 C3 supper mini
Parts:
- removed BUT1: TS-1187A-B-A-B, Button_Switch_SMD:SW_SPST_TL3342, symbol TS-1187A-B-A-B
- removed C10: 4.7nF, Capacitor_SMD:C_0805_2012Metric, symbol 0603B472K500NT
- removed C11: 100nF, Capacitor_SMD:C_0805_2012Metric, symbol CC0603KRX7R9BB104_9
- removed C12: 100nF, Capacitor_SMD:C_0805_2012Metric, symbol CC0603KRX7R9BB104
- removed C17: 10nF, Capacitor_SMD:C_0805_2012Metric, symbol 0603B103K500NT_1
- removed C18: 100nF, Capacitor_SMD:C_0805_2012Metric, symbol CC0603KRX7R9BB104_3
- removed C19: 4.7uF, Capacitor_SMD:C_0805_2012Metric, symbol 1206B475K500NT_1
- removed C2: 10nF, Capacitor_SMD:C_0805_2012Metric, symbol 0603B103K500NT_2
- removed C20: 4.7uF, Capacitor_SMD:C_0805_2012Metric, symbol 1206B475K500NT
- removed C21: 100nF, Capacitor_SMD:C_0805_2012Metric, symbol CC0603KRX7R9BB104_2
- removed C22: 10nF, Capacitor_SMD:C_0805_2012Metric, symbol 0603B103K500NT
- removed C3: 4.7uF, Capacitor_SMD:C_0805_2012Metric, symbol 1206B475K500NT_4
- removed C4: 10uF, Capacitor_SMD:C_1206_3216Metric, symbol CL10A106KP8NNNC_1
- removed C42: 18pF, Capacitor_SMD:C_0805_2012Metric, symbol CL10C180JB8NNNC
- removed C43: 18pF, Capacitor_SMD:C_0805_2012Metric, symbol CL10C180JB8NNNC_1
- removed C44: 4.7uF, Capacitor_SMD:C_0805_2012Metric, symbol CL10A475KO8NNNC
- removed C46: 100nF, Capacitor_SMD:C_0805_2012Metric, symbol CC0603KRX7R9BB104_12
- removed C47: 4.7uF, Capacitor_SMD:C_0805_2012Metric, symbol CL10A475KO8NNNC_1
- removed C49: 4.7uF, Capacitor_SMD:C_0805_2012Metric, symbol CL10A475KO8NNNC_3
- removed C50: 100nF, Capacitor_SMD:C_0805_2012Metric, symbol CC0603KRX7R9BB104_13
- removed C51: 100nF, Capacitor_SMD:C_0805_2012Metric, symbol CC0603KRX7R9BB104_14
- removed C52: 4.7uF, Capacitor_SMD:C_0805_2012Metric, symbol CL10A475KO8NNNC_4
- removed C53: 100nF, Capacitor_SMD:C_0805_2012Metric, symbol CC0603KRX7R9BB104_15
- removed C54: 4.7uF, Capacitor_SMD:C_0805_2012Metric, symbol CL10A475KO8NNNC_5
- removed C6: 10uF, Capacitor_SMD:C_1206_3216Metric, symbol CL10A106KP8NNNC
- removed C7: 100nF, Capacitor_SMD:C_0805_2012Metric, symbol CC0603KRX7R9BB104_1
- removed H2: KH-2.54PH180-1X7P-L11.5, Connector_PinHeader_2.54mm:PinHeader_1x07_P2.54mm_Vertical, symbol KH-2.54PH180-1X7P-L11.5
- removed H3: KH-2.54PH180-1X7P-L11.5, Connector_PinHeader_2.54mm:PinHeader_1x07_P2.54mm_Vertical, symbol KH-2.54PH180-1X7P-L11.5_1
- removed H5: KH-2.54PH180-1X7P-L11.5, Connector_PinHeader_2.54mm:PinHeader_1x07_P2.54mm_Vertical, symbol KH-2.54PH180-1X7P-L11.5_2
- removed J-LINK1: 20021111-00010T4LF, Connector_PinHeader_2.54mm:PinHeader_2x05_P2.54mm_Vertical, symbol 20021111-00010T4LF
- removed L3: 470Ω, Inductor_SMD:L_1210_3225Metric, symbol BLM18PG471SN1D
- removed LED1: 19-217/GHC-YR1S2/3T, LED_SMD:LED_0805_2012Metric, symbol 19-217/GHC-YR1S2/3T
- removed R1: 27kΩ, Resistor_SMD:R_0805_2012Metric, symbol 0603WAF2702T5E
- removed R10: 100Ω, Resistor_SMD:R_0805_2012Metric, symbol 0603WAF1000T5E_3
- removed R16: 100kΩ, Resistor_SMD:R_0805_2012Metric, symbol 0603WAF1003T5E_1
- removed R2: 5.1kΩ, Resistor_SMD:R_0805_2012Metric, symbol 0603WAF5101T5E
- removed R3: 47kΩ, Resistor_SMD:R_0805_2012Metric, symbol 0603WAF4702T5E
- removed R38: 0Ω, Resistor_SMD:R_0805_2012Metric, symbol 0603WAF0000T5E
- removed R4: 1kΩ, Resistor_SMD:R_0805_2012Metric, symbol 0603WAF1001T5E_5
- removed R40: 1kΩ, Resistor_SMD:R_0805_2012Metric, symbol 0603WAF1001T5E_6
- removed R43: 1kΩ, Resistor_SMD:R_0805_2012Metric, symbol 0603WAF1001T5E_13
- removed R44: 1kΩ, Resistor_SMD:R_0805_2012Metric, symbol 0603WAF1001T5E_11
- removed R45: 1kΩ, Resistor_SMD:R_0805_2012Metric, symbol 0603WAF1001T5E_9
- removed R46: 1kΩ, Resistor_SMD:R_0805_2012Metric, symbol 0603WAF1001T5E_8
- removed R47: 1kΩ, Resistor_SMD:R_0805_2012Metric, symbol 0603WAF1001T5E_14
- removed R48: 1kΩ, Resistor_SMD:R_0805_2012Metric, symbol 0603WAF1001T5E_12
- removed R49: 1kΩ, Resistor_SMD:R_0805_2012Metric, symbol 0603WAF1001T5E_15
- removed R50: 1kΩ, Resistor_SMD:R_0805_2012Metric, symbol 0603WAF1001T5E_18
- removed R51: 1kΩ, Resistor_SMD:R_0805_2012Metric, symbol 0603WAF1001T5E_19
- removed R52: 1kΩ, Resistor_SMD:R_0805_2012Metric, symbol 0603WAF1001T5E_10
- removed R53: 1kΩ, Resistor_SMD:R_0805_2012Metric, symbol 0603WAF1001T5E_17
- removed R54: 1kΩ, Resistor_SMD:R_0805_2012Metric, symbol 0603WAF1001T5E_16
- removed R6: 1MΩ, Resistor_SMD:R_0805_2012Metric, symbol 0603WAF1004T5E
- removed R7: 5.1kΩ, Resistor_SMD:R_0805_2012Metric, symbol 0603WAF5101T5E_1
- removed TP16: 1-POINT TEST POINT, TestPoint:TestPoint_Pad_D1.5mm, symbol 1-POINT TEST POINT_13
- removed TP17: 1-POINT TEST POINT, TestPoint:TestPoint_Pad_D1.5mm, symbol 1-POINT TEST POINT_14
- removed TP3: 1-POINT TEST POINT, TestPoint:TestPoint_Pad_D1.5mm, symbol 1-POINT TEST POINT_2
- removed TP4: 1-POINT TEST POINT, TestPoint:TestPoint_Pad_D1.5mm, symbol 1-POINT TEST POINT_3
- removed TP5: 1-POINT TEST POINT, TestPoint:TestPoint_Pad_D1.5mm, symbol 1-POINT TEST POINT_4
- removed U1: ESP32-C3-SuperMini, Connector_PinHeader_2.54mm:PinHeader_2x08_P2.54mm_Vertical, symbol ESP32-C3-SuperMini
- removed U9: MF-ASML020/6-2, Package_SO:SOIC-8_3.9x4.9mm_P1.27mm, symbol MF-ASML020/6-2
- removed USBC1: USB3.1C16PFSMT, Connector_USB:USB_C_Receptacle_HRO_TYPE-C-31-M-12, symbol USB3.1C16PFSMT
- removed X1: 32.768kHz, Crystal:Crystal_SMD_3225-4Pin_3.2x2.5mm, symbol Q13FC1350000400
- added U16: ESP32-C3_SUPERMINI_TH, bGeigieScint:MODULE_ESP32-C3_SUPERMINI_TH, symbol ESP32-C3_SUPERMINI_TH:ESP32-C3_SUPERMINI_TH
Connections:
- net 3V3: now also C48.2, U16.3.3 (3V3)
- net GND: now also U16.G (GND)
- net PA16_SDA: now also U16.8 (GPIO8)
- net PA17_SCL: now also U16.9 (GPIO9)
- no-connect marks 15 -> 9
Other:
- note removed: "3V3"
- moved on the sheet: C48, C55, C56, D1, D9, P1, P2, Q3, R37, R39, TP12, TP13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
