File: bGeigieScint/bGeigieScint.kicad_sch (KiCad schematic)
At the start: 112 parts, among them P1 Header-Male-2.54_2x2, P2 Header-Male-2.54_2x2, Q1 BC847_C2910145, Q2 MMBT5551LT1G, Q3 AO3401A, Q4 AO3401A, Q5 MMBT5551LT1G, U10 74LVC1G08GV,125, U11 LT3014BHVES5#TRMPBF, U12 TXU0202DCUR, U13 TLV7031DBVR, U14 TLR341G-GTR, U15 803-87-006-10-001101, U16 ESP32-C3_SUPERMINI_TH, U2 XC6209F332MR-G, U3 MC14043BDR2G, U4 LMV793MFX/NOPB, U5 TPS7A2030PDBVR, U6 TLV3201AIDBVT, U7 OPA357AIDBVR, U8 TLR341G-GTR

Commit message: Cleaned up
Parts:
- removed C45: 1uF, Capacitor_SMD:C_0805_2012Metric, symbol CL10A105KB8NNNC_4
- removed TP10: 1-POINT TEST POINT, TestPoint:TestPoint_Pad_D1.5mm, symbol 1-POINT TEST POINT_8
- removed TP11: 1-POINT TEST POINT, TestPoint:TestPoint_Pad_D1.5mm, symbol 1-POINT TEST POINT_9
- removed TP12: 1-POINT TEST POINT, TestPoint:TestPoint_Pad_D1.5mm, symbol 1-POINT TEST POINT_15
- removed TP13: 1-POINT TEST POINT, TestPoint:TestPoint_Pad_D1.5mm, symbol 1-POINT TEST POINT_10
- removed TP14: 1-POINT TEST POINT, TestPoint:TestPoint_Pad_D1.5mm, symbol 1-POINT TEST POINT_11
- removed TP15: 1-POINT TEST POINT, TestPoint:TestPoint_Pad_D1.5mm, symbol 1-POINT TEST POINT_12
- removed TP18: 1-POINT TEST POINT, TestPoint:TestPoint_Pad_D1.5mm, symbol 1-POINT TEST POINT_17
- removed TP6: 1-POINT TEST POINT, TestPoint:TestPoint_Pad_D1.5mm, symbol 1-POINT TEST POINT_5
- removed TP7: 1-POINT TEST POINT, TestPoint:TestPoint_Pad_D1.5mm, symbol 1-POINT TEST POINT_6
- removed TP8: 1-POINT TEST POINT, TestPoint:TestPoint_Pad_D1.5mm, symbol 1-POINT TEST POINT_16
- removed TP9: 1-POINT TEST POINT, TestPoint:TestPoint_Pad_D1.5mm, symbol 1-POINT TEST POINT_7
Other:
- moved on the sheet: C1, C13, C14, C15, C16, C23, C24, C25, C26, C27, C28, C29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

Commit message: refactor: Remove unused schematic symbol definitions, add a 3D model, and update KiCad schematic and PCB files.
Parts:
- removed C56: 100nF, Capacitor_SMD:C_0805_2012Metric, symbol CC0603KRX7R9BB104_17
- removed R39: 27kΩ, Resistor_SMD:R_0805_2012Metric, symbol 0603WAF2702T5E_1
- removed U12: TXU0202DCUR, Package_SO:VSSOP-8_2.3x2mm_P0.5mm, symbol TXU0202DCUR
- removed U15: 803-87-006-10-001101, Connector_PinSocket_2.54mm:PinSocket_1x06_P2.54mm_Vertical, symbol 803-87-006-10-001101
Other:
- moved on the sheet: C13, C14, C15, C16, C24, C30, C34, C35, C36, C37, C55, C9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
