File: bGeigieScint/bGeigieScint.kicad_sch (KiCad schematic)
At the start: 96 parts, among them P1 Header-Male-2.54_2x2, P2 Header-Male-2.54_2x2, Q1 BC847_C2910145, Q2 MMBT5551LT1G, Q3 AO3401A, Q4 AO3401A, Q5 MMBT5551LT1G, U10 74LVC1G08GV,125, U11 LT3014BHVES5#TRMPBF, U13 TLV7031DBVR, U14 TLR341G-GTR, U16 ESP32-C3_SUPERMINI_TH, U2 XC6209F332MR-G, U3 MC14043BDR2G, U4 LMV793MFX/NOPB, U5 TPS7A2030PDBVR, U6 TLV3201AIDBVT, U7 OPA357AIDBVR, U8 TLR341G-GTR

Commit message: Added 3d model files, how to build files, etc
Other:
- moved on the sheet: C1, C13, C14, C15, C16, C23, C24, C25, C26, C27, C28, C29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
