File: bGeigieScint/bGeigieScint.kicad_pcb (KiCad board)
At the start: 4 copper layers, 38.1 x 66 mm, 112 parts, among them P1 Header-Male-2.54_2x2, P2 Header-Male-2.54_2x2, Q1 BC847_C2910145, Q2 MMBT5551LT1G, Q3 AO3401A, Q4 AO3401A, Q5 MMBT5551LT1G, U10 74LVC1G08GV,125, U11 LT3014BHVES5#TRMPBF, U12 TXU0202DCUR, U13 TLV7031DBVR, U14 TLR341G-GTR, U15 803-87-006-10-001101, U16 ESP32-C3_SUPERMINI_TH, U2 XC6209F332MR-G, U3 MC14043BDR2G, U4 LMV793MFX/NOPB, U5 TPS7A2030PDBVR, U6 TLV3201AIDBVT, U7 OPA357AIDBVR, U8 TLR341G-GTR

Commit message: Cleaned up
Parts:
- removed C45: 1uF, Capacitor_SMD:C_0805_2012Metric
- removed TP10, TP11, TP12, TP13, TP14, TP15, TP18, TP6, TP7, TP8, TP9: 1-POINT TEST POINT, TestPoint:TestPoint_Pad_D1.5mm
Connections:
- MEAS1 pad 2: Net-(MEAS1-Pad2) -> unconnected-(MEAS1-Pad2)
