File: bGeigieScint/bGeigieScint.kicad_pcb (KiCad board)
At the start: 4 copper layers, 38.1 x 66 mm, 100 parts, among them P1 Header-Male-2.54_2x2, P2 Header-Male-2.54_2x2, Q1 BC847_C2910145, Q2 MMBT5551LT1G, Q3 AO3401A, Q4 AO3401A, Q5 MMBT5551LT1G, U10 74LVC1G08GV,125, U11 LT3014BHVES5#TRMPBF, U12 TXU0202DCUR, U13 TLV7031DBVR, U14 TLR341G-GTR, U15 803-87-006-10-001101, U16 ESP32-C3_SUPERMINI_TH, U2 XC6209F332MR-G, U3 MC14043BDR2G, U4 LMV793MFX/NOPB, U5 TPS7A2030PDBVR, U6 TLV3201AIDBVT, U7 OPA357AIDBVR, U8 TLR341G-GTR

Commit message: Add Projet Luciole reference project, Polemo Core 2 schematic, and KiCad updates
- Import luciole/ (Projet Luciole scintillation spectrometer: electronics, firmware, docs, mech)
- Rename autosave to Polemo Core 2.kicad_sch
- Update bGeigieScint PCB and project files
- Add crystal handling/storage guide PDF and KiCad backups
- Ignore bGeigieScint/.history/ editor local-history

Co-Authored-By: Claude Fable 5 <noreply@anthropic.com>
Other:
- board text added: "bGeigieScint Sensor-board V0.9B"
Changed lines of the file:
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@@
 		(layer "Edge.Cuts")
 	)
-	(gr_text ""
-		(at 5 5 0)
-		(layer "Dwgs.User")
+	(gr_text "bGeigieScint\nSensor-board V0.9B"
+		(at 100 145 0)
+		(layer "F.Silkscreen")
 		(effects
 			(font
-				(size 10 10)
-				(thickness 1)
+				(size 1.5 1.5)
+				(thickness 0.25)
 			)
 			(justify left top)
