File: Open_Gamma_Detector/hardware/PCB_Project_EasyEDA.kicad_pcb (KiCad board)
At the start: 4 copper layers, 120 x 50 mm, 71 parts, among them Q1 2N7002,215, Q2 2N7002,215, SW1 TSC015A03526A, U1 TLV3201AIDBVR, U2 LM4040AIM3-3.0+T, U3 RASPBERRY PI PICO 2, U4 OPA357AIDBVR, U5 MAX5026EUT+T, U6 LM4040AIM3-3.0+T, U7 OPA357AIDBVR, U8 OPA357AIDBVR

Commit message: This version of Antigravity is no longer supported. Please update to receive the latest features!
Changed lines of the file:
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@@
 		(embedded_fonts no)
 		(model "${KIPRJMOD}/EASYEDA_MODELS/PICO.step"
+			(hide yes)
 			(offset
 				(xyz -10.5 -25.5501 1.6)
@@
 			)
 		)
+		(model "${KIPRJMOD}/EASYEDA_MODELS/Raspberry Pi Pico-R3.STEP"
+			(offset
+				(xyz 0 0 0)
+			)
+			(scale
+				(xyz 1 1 1)
+			)
+			(rotate
+				(xyz -90 -0 -0)
+			)
+		)
 	)
 	(footprint "C0805"
@@
 					(face "NotoSerifCJKsc-Medium")
 					(size 0.9144 0.9144)
-					(thickness 0.254)
+					(thickness 0.2286)
 				)
 				(justify left top)
@@
 		(model "${KIPRJMOD}/EASYEDA_MODELS/HDR-TH_4P-P2.54-F-LI-1X4P.step"
 			(offset
-				(xyz 0 -0 -3)
+				(xyz 0 -0 0)
 			)
 			(scale
@@
 			)
 			(rotate
-				(xyz -0 -0 0)
+				(xyz -0 -0 -0)
 			)
 		)
@@
 		(model "${KIPRJMOD}/EASYEDA_MODELS/HDR-TH_10P-P2.54-F-LI-1X10P.step"
 			(offset
-				(xyz -0 -0 -3.3)
+				(xyz -0 -0 4.2)
 			)
 			(scale
@@
 			)
 			(rotate
-				(xyz -0 -0 0)
+				(xyz -0 -0 -0)
 			)
 		)
